File: socketboard.kicad_sch (KiCad schematic)
At the start: 11 parts, among them J1 GPIO, J2 Conn_01x07, J3 Conn_01x03, U1 MCP2518FDT-H/SL, U2 ATA6563-GBQW1, Y1 Oscillator

Commit message: final
Parts:
- removed Y1: Oscillator, Oscillator:Oscillator_SMD_Diodes_FN-4Pin_7.0x5.0mm, symbol PCM_SparkFun-Clock:Oscillator
- added C5: 4.7uF, PCM_SparkFun-Capacitor:C_0603_1608Metric, symbol PCM_SparkFun-Capacitor:C_Small
- added R2: 10k, PCM_SparkFun-Resistor:R_0603_1608Metric, symbol PCM_SparkFun-Resistor:R_Small
- added R3: 4.7k, PCM_SparkFun-Resistor:R_0603_1608Metric, symbol PCM_SparkFun-Resistor:R_Small
- added Y2: SG-210STF, Oscillator:Oscillator_SMD_SeikoEpson_SG210-4Pin_2.5x2.0mm, symbol Oscillator:SG-210STF
- J2: footprint PCM_SparkFun-Connector:1x07_P2.54mm -> Connector_PinSocket_2.54mm:PinSocket_1x07_P2.54mm_Vertical
- J3: footprint Connector_PinHeader_2.54mm:PinHeader_1x03_P2.54mm_Vertical -> Connector_PinSocket_2.54mm:PinSocket_1x03_P2.54mm_Vertical
Connections:
- net 3.3V: now also C1.2, C5.1, R2.2, Y2.1 (~{ST}), Y2.4 (Vcc); no longer C1.1
- net CANH: now also R1.2
- net CANL: now also R1.1
- net GND: now also C1.1, C5.2, R3.2, Y2.2 (GND); no longer C1.2, U2.8 (STBY)
- net GPIO8/SPI0.CE0: now also U1.13 (NCS); no longer U1.4 (*INT)
- net OSC1: now also Y2.3 (OUT)
- net RXD: no longer R1.2
- net TXD: no longer R1.1
- net STBY: now reaches U1.9 (*INT0/GPIO0/XSTBY)
- net STBY: now also U2.8 (STBY), R3.1
- net GPIO25: now reaches J1.22 (Pin_22)
- net GPIO25: now also U1.4 (*INT), R2.1
- no-connect marks 27 -> 26
Other:
- note added: "GPIO Pull up"
- moved on the sheet: C2, J3
